Commit message: simulation_ws for TheConstruct + Melodic + Turtlebot

File: src/turtlebot/kobuki_description/urdf/kobuki.urdf.xacro (robot description, xacro)
@@ -228,5 +228,5 @@
 		    <origin xyz="0 0 0" rpy="0 0 0"/>
 		    <geometry>
-			    <mesh filename="package://hokuyo/meshes/hokuyo.dae"/>
+			    <mesh filename="package://gazebo_plugins/test/multi_robot_scenario/meshes/laser/hokuyo.dae"/>
 		    </geometry>
 	    </visual>

File: src/turtlebot/kobuki_description/urdf/kobuki_gazebo.urdf.xacro (robot description, xacro)
@@ -175,8 +175,14 @@
 	    <publishWheelJointState>true</publishWheelJointState>
 	    <legacyMode>true</legacyMode>
+	    <rosDebugLevel>na</rosDebugLevel>
+	    <publishWheelTF>false</publishWheelTF>
+        <wheelAcceleration>0</wheelAcceleration>
+        <wheelTorque>5</wheelTorque>
+        <odometrySource>world</odometrySource>
+        <publishTf>1</publishTf>
 	  </plugin>
 	</gazebo>
 	<gazebo reference="laser_sensor_link">
-		<sensor type="gpu_ray" name="laser_sensor">
+		<sensor type="ray" name="laser_sensor">
 			<pose>0 0 0 0 0 0</pose>
 			<visualize>false</visualize>
@@ -202,5 +208,5 @@
 				</noise>
 			</ray>
-			<plugin name="gazebo_ros_head_hokuyo_controller" filename="libgazebo_ros_gpu_laser.so">
+			<plugin name="gazebo_ros_head_hokuyo_controller" filename="libgazebo_ros_laser.so">
 				<topicName>/kobuki/laser/scan</topicName>
 				<frameName>laser_sensor_link</frameName>
