Commit message: first cleanup for noetic

File: larm/urdf/kobuki_car.urdf.xacro (robot description, xacro)
@@ -34,5 +34,5 @@
         <origin xyz="0.001 0 0.05199" rpy="0 0 0"/>
       </visual>
-      <collision>
+      <collision name="base">
         <geometry>
           <cylinder length="0.10938" radius="0.178"/>
@@ -71,5 +71,5 @@
       <collision>
         <geometry>
-          <cylinder length="0.0206" radius="0.0352"/>
+          <cylinder length="0.0206" radius="0.035"/>
         </geometry>
         <origin rpy="0 0 0" xyz="0 0 0"/>
@@ -98,5 +98,5 @@
       <collision>
         <geometry>
-          <cylinder length="0.0206" radius="0.0350"/>
+          <cylinder length="0.0206" radius="0.035"/>
         </geometry>
         <origin rpy="0 0 0" xyz="0 0 0"/>
@@ -234,5 +234,5 @@
     </link>
     <!-- Kobuki Gazebo simulation details -->
-    <kobuki_sim/>
+    <xacro:kobuki_sim/>
   </xacro:macro>
 </robot>

File: larm/urdf/turtlebot_car.urdf.xacro (robot description, xacro)
@@ -3,20 +3,13 @@
     - Base      : kobuki
     - Stacks    : hexagons
-    - 3d Sensor : asus xtion pro
-    - hokuyo
+    - 3d Sensor : kinect
 -->
-<robot name="turtlebot" xmlns:xacro="http://ros.org/wiki/xacro">
-  <!-- General -->
-  <xacro:include filename="$(find turtlebot_description)/urdf/common_properties.urdf.xacro"/>
-  <xacro:include filename="$(find turtlebot_description)/urdf/turtlebot_properties.urdf.xacro"/>
-  <!-- Bases -->
+<robot name="turtlebot_car" xmlns:xacro="http://ros.org/wiki/xacro">
+  <xacro:include filename="$(find turtlebot_description)/urdf/turtlebot_common_library.urdf.xacro" />
   <xacro:include filename="$(find larm)/urdf/kobuki_car.urdf.xacro" />
-  <!-- Stacks -->
-  <xacro:include filename="$(find larm)/urdf/car.urdf.xacro"/>
-  <!-- 3D Sensors -->
-  <xacro:include filename="$(find kobuki_description)/urdf/sensors/kinect.urdf.xacro"/>
-  <xacro:include filename="$(find kobuki_description)/urdf/sensors/asus_xtion_pro.urdf.xacro"/>
-  <kobuki_car/>
-  <stack_hexagons                 parent="base_link"/>
-  <sensor_asus_xtion_pro          parent="base_link"/>
+  <xacro:include filename="$(find larm)/urdf/hexagons_car.urdf.xacro"/>
+  <xacro:include filename="$(find turtlebot_description)/urdf/sensors/xtion_pro.urdf.xacro"/>
+  <xacro:kobuki_car/>
+  <xacro:stack_hexagons   parent="base_link"/>
+  <xacro:sensor_xtion_pro parent="base_link" xtion_pro_cam_py="0.0205"/>
 </robot>
